File: PLC Arduino/PLC Arduino-backups/PLC Arduino-2024-08-29_035323/PLC Arduino.kicad_sch (KiCad schematic)
At the start: 188 parts, among them J1 Screw_Terminal_01x12, J10 Conn_01x02_Socket, J2 Screw_Terminal_01x12, J3 Screw_Terminal_01x12, J4 Screw_Terminal_01x12, J5 USB_B_Micro, J6 Conn_01x04_Socket, J7 Conn_01x03_Socket, J8 Conn_01x02_Socket, J9 Conn_01x02_Socket, K1 Y14x-1C-xxDS, K2 Y14x-1C-xxDS, K3 Y14x-1C-xxDS, K4 Y14x-1C-xxDS, Q1 Q_NMOS_Depletion_GSD, Q10 BSS138, Q2 Q_NMOS_Depletion_GSD, Q3 Q_NMOS_Depletion_GSD, Q4 Q_NMOS_Depletion_GSD, Q5 Q_NMOS_Depletion_GSD, Q6 Q_NMOS_Depletion_GSD, Q7 Q_NMOS_Depletion_GSD, Q8 Q_NMOS_Depletion_GSD, Q9 BSS138, SW1 SW_Push, SW2 SW_Push, U1 PC817, U10 PC817, U11 PC817, U12 PC817, U13 PC817, U14 PC817, U15 PC817, U16 PC817, U17 OP07, U18 ADS1115IDGS, U19 OP07, U2 PC817, U20 OP07, U21 OP07, U22 ISO1540, U23 ESP32-WROOM-32, U24 CH340C, U25 MAX485E, U26 MAX485E, U27 TPL5010, U28 LM2596S-5, U29 AMS1117-3.3, U3 PC817, U32 LM2596S-12, U4 PC817, U5 PC817, U6 PC817, U7 PC817, U8 PC817, U9 PC817

Commit message: Updated PLC Arduino Project
Added Power Isolation and Pin Mapping
Parts:
- removed C21: 10uF, Capacitor_SMD:C_0805_2012Metric_Pad1.18x1.45mm_HandSolder, symbol Device:C
- removed C22: 0.1uF, Capacitor_SMD:C_0402_1005Metric, symbol Device:C
- removed C23, C28: 100uF, Capacitor_SMD:C_Elec_10x10.2, symbol Device:C_Polarized
- removed C24, C29: 220uF, Capacitor_SMD:C_Elec_6.3x7.7, symbol Device:C_Polarized
- removed C25, C30: 1000uF, Capacitor_SMD:C_Elec_10x10.2, symbol Device:C_Polarized
- removed C26, C27: 22uF, Capacitor_SMD:C_0603_1608Metric, symbol Device:C_Polarized
- removed D15, D17: SS54, Diode_SMD:D_SMA, symbol Diode:1N4001
- removed D16, D18: LED, LED_SMD:LED_0805_2012Metric_Pad1.15x1.40mm_HandSolder, symbol Device:LED
- removed J10, J8: Conn_01x02_Socket, Connector_PinHeader_2.54mm:PinHeader_1x02_P2.54mm_Vertical, symbol Connector:Conn_01x02_Socket
- removed J9: Conn_01x02_Socket, Connector_JST:JST_PH_B2B-PH-K_1x02_P2.00mm_Vertical, symbol Connector:Conn_01x02_Socket
- removed L1, L2: 33uH, Inductor_SMD:L_Chilisin_BMRF00101040, symbol Device:L
- removed R67, R68: 1K, Resistor_SMD:R_0603_1608Metric, symbol Device:R
- removed U28: LM2596S-5, Package_TO_SOT_SMD:TO-263-5_TabPin3, symbol Regulator_Switching:LM2596S-5
- removed U29: AMS1117-3.3, Package_TO_SOT_SMD:SOT-223-3_TabPin2, symbol Regulator_Linear:AMS1117-3.3
- removed U32: LM2596S-12, Package_TO_SOT_SMD:TO-263-5_TabPin3, symbol Regulator_Switching:LM2596S-12
Connections:
- net +24V: no longer J2.12 (Pin_12)
- net +3.3V: no longer U22.8 (VCC2)
- net 3.3VOUT: no longer J2.10 (Pin_10), J4.9 (Pin_9)
- net 5VOUT: no longer J2.11 (Pin_11), J4.10 (Pin_10)
- net GND: no longer J2.7 (Pin_7), J2.8 (Pin_8), J2.9 (Pin_9), J4.6 (Pin_6)
- net GNDD: no longer U22.5 (GND2)
- net SCL: no longer J4.7 (Pin_7)
- net SDA: no longer J4.8 (Pin_8)
- net ESP_SCL: no longer names the net of U23.36 (IO22)
- net ESP_SCL: no longer U22.6 (SCL2)
- net ESP_SDA: no longer names the net of U23.33 (IO21)
- net ESP_SDA: no longer U22.7 (SDA2)
Other:
- note removed: "POWER SUPPLY"
