File: PLC Arduino/PLC Arduino.kicad_sch (KiCad schematic)
At the start: 164 parts, among them J1 Screw_Terminal_01x12, J2 Screw_Terminal_01x12, J3 Screw_Terminal_01x12, J4 Screw_Terminal_01x12, J5 USB_B_Micro, J6 Conn_01x04_Socket, J7 Conn_01x03_Socket, K1 Y14x-1C-xxDS, K2 Y14x-1C-xxDS, K3 Y14x-1C-xxDS, K4 Y14x-1C-xxDS, Q1 Q_NMOS_Depletion_GSD, Q10 BSS138, Q2 Q_NMOS_Depletion_GSD, Q3 Q_NMOS_Depletion_GSD, Q4 Q_NMOS_Depletion_GSD, Q5 Q_NMOS_Depletion_GSD, Q6 Q_NMOS_Depletion_GSD, Q7 Q_NMOS_Depletion_GSD, Q8 Q_NMOS_Depletion_GSD, Q9 BSS138, SW1 SW_Push, SW2 SW_Push, U1 PC817, U10 PC817, U11 PC817, U12 PC817, U13 PC817, U14 PC817, U15 PC817, U16 PC817, U17 OP07, U18 ADS1115IDGS, U19 OP07, U2 PC817, U20 OP07, U21 OP07, U22 ISO1540, U23 ESP32-WROOM-32, U24 CH340C, U25 MAX485E, U26 MAX485E, U27 TPL5010, U3 PC817, U4 PC817, U5 PC817, U6 PC817, U7 PC817, U8 PC817, U9 PC817

Commit message: Updated PLC Arduino Project
Added Power Isolation and Pin Mapping
Parts:
- added C21, C25, C32, C34, C36: 10uF, Capacitor_SMD:C_0805_2012Metric_Pad1.18x1.45mm_HandSolder, symbol Device:C
- added C22: 100uF, Capacitor_SMD:C_Elec_10x10.2, symbol Device:C_Polarized
- added C23, C26: 100uF, Capacitor_SMD:C_0805_2012Metric_Pad1.18x1.45mm_HandSolder, symbol Device:C
- added C24: 220uF, Capacitor_SMD:C_Elec_6.3x7.7, symbol Device:C_Polarized
- added C27: 1000uF, Capacitor_SMD:C_Elec_10x10.2, symbol Device:C_Polarized
- added C28, C29: 22uF, Capacitor_SMD:C_0603_1608Metric, symbol Device:C_Polarized
- added C30, C31: 22uF, Capacitor_SMD:C_0805_2012Metric_Pad1.18x1.45mm_HandSolder, symbol Device:C
- added C33, C35, C37: 0.1uF, Capacitor_SMD:C_0402_1005Metric, symbol Device:C
- added D15: SS54, Diode_SMD:D_SMA, symbol Diode:1N4001
- added D16: LED, LED_SMD:LED_0805_2012Metric_Pad1.15x1.40mm_HandSolder, symbol Device:LED
- added J8: Conn_01x02_Socket, Connector_PinHeader_2.54mm:PinHeader_1x02_P2.54mm_Vertical, symbol Connector:Conn_01x02_Socket
- added J9: Conn_01x02_Socket, Connector_JST:JST_PH_B2B-PH-K_1x02_P2.00mm_Vertical, symbol Connector:Conn_01x02_Socket
- added L1: 33uH, Inductor_SMD:L_Chilisin_BMRF00101040, symbol Device:L
- added R67: 1K, Resistor_SMD:R_0603_1608Metric, symbol Device:R
- added U28: B0505S-2WR3, B_S-2WR2_MNS, symbol 2024-08-29_08-56-51:B0505S-2WR3
- added U29: LM2596S-5, Package_TO_SOT_SMD:TO-263-5_TabPin3, symbol Regulator_Switching:LM2596S-5
- added U30, U31: AMS1117-3.3, Package_TO_SOT_SMD:SOT-223-3_TabPin2, symbol Regulator_Linear:AMS1117-3.3
- added U32, U33: 74HC595, Package_SO:SOIC-16_3.9x9.9mm_P1.27mm, symbol 74xx:74HC595
- added U34: 74HC4051, symbol 74xx:74HC4051
Connections:
- net +24V: now also C22.1, U29.1 (VIN)
- net +3.3V: now also U22.8 (VCC2), C31.2, C32.2, C33.1, U31.2 (VO)
- net +3.3VA: now also C29.1, U30.2 (VO)
- net +5V: now also C25.2, C26.2, C30.2, C34.2, C35.2, C36.2, C37.2, U28.6 (+VO), U31.3 (VI), U32.10 (~{SRCLR}), U32.16 (VCC), U33.10 (~{SRCLR}), U33.16 (VCC), U34.16 (VCC)
- net +5VA: now also C21.2, C23.2, C24.1, C27.1, C28.1, J8.2 (Pin_2), L1.2, R67.1, U28.1 (VIN), U30.3 (VI)
- net 24VIN: now also J2.12 (Pin_12)
- net 3.3VOUT: now also J2.10 (Pin_10), J4.9 (Pin_9)
- net 5VOUT: now also J2.11 (Pin_11), J4.10 (Pin_10)
- net DC_DRV_1: now also U32.4 (QE)
- net DC_DRV_2: now also U32.5 (QF)
- net DC_DRV_3: now also U32.6 (QG)
- net DC_DRV_4: now also U32.7 (QH)
- net DOUT_DRV_1: now also U32.15 (QA)
- net DOUT_DRV_2: now also U32.1 (QB)
- net DOUT_DRV_3: now also U32.2 (QC)
- net DOUT_DRV_4: now also U32.3 (QD)
- net GND: now also J2.7 (Pin_7), J2.8 (Pin_8), J2.9 (Pin_9), J4.6 (Pin_6)
- net GNDD: now also U22.5 (GND2), C25.1, C26.1, C34.1, C35.1, C36.1, C37.1, U28.4 (0V), U32.13 (~{OE}), U32.8 (GND), U33.13 (~{OE}), U33.8 (GND), U34.7 (VEE), U34.8 (GND)
- net GNDPWR: now also C21.1, C22.2, C23.1, C24.2, C27.2, C28.2, C29.2, C30.1, C31.1, C32.1, C33.2, D15.2 (A), D16.1 (K), J9.2 (Pin_2), U28.2 (GND), U29.3 (GND), U29.5 (~{ON}/OFF), U30.1 (GND), U31.1 (GND)
- net MASTER_DI: now also U23.27 (IO16)
- net MASTER_EN: now also U23.23 (IO15)
- net MASTER_RO: now also U23.28 (IO17)
- net SCL: now also J4.7 (Pin_7)
- net SDA: now also J4.8 (Pin_8)
- net SLAVE_DI: now also U23.16 (IO13)
- net SLAVE_EN: now also U23.26 (IO4)
- net SLAVE_RO: now also U23.13 (IO14)
- net WDT_DONE: now also U23.30 (IO18), U27.4 (DONE)
- net REG_CLK: now reaches U23.10 (IO25)
- net REG_CLK: now also U32.11 (SRCLK), U33.11 (SRCLK)
- net REG_CS: now reaches U23.11 (IO26)
- net REG_CS: now also U32.12 (RCLK), U33.12 (RCLK)
- net DIG_IN: now reaches U23.31 (IO19)
- net DIG_IN: now also U34.3 (A)
- net ESP_SDA: now reaches U23.33 (IO21)
- net ESP_SDA: now also U22.7 (SDA2)
- net ESP_SCL: now reaches U23.36 (IO22)
- net ESP_SCL: now also U22.6 (SCL2)
- net REG_DIN: now reaches U23.37 (IO23)
- net REG_DIN: now also U32.14 (SER)
- new net: D16.2 (A), J9.1 (Pin_1), R67.2
- new net: D15.1 (K), L1.1, U29.2 (OUT)
- new net: J8.1 (Pin_1), U29.4 (FB)
- new net: U32.9 (QH'), U33.14 (SER)
- new net MUX_EN: U33.3 (QD), U34.6 (~{E})
- new net MUX_S0: U33.15 (QA), U34.11 (S0)
- new net MUX_S1: U33.1 (QB), U34.10 (S1)
- new net MUX_S2: U33.2 (QC), U34.9 (S2)
- no-connect marks 22 -> 24
Other:
- note added: "5V ISOLATION"
- note added: "INPUT MONITOR"
- note added: "OUTPUT CONTROL"
- note added: "Output Capacity 5V, 400mA"
- note added: "POWER SUPPLY"
- moved on the sheet: C10, C11, C12, C13, C9, R50, SW1, SW2, U23

Commit message: Added Mapping for Inputs to MUX
Connections:
- net DC_IN_1: now also U34.13 (A0)
- net DC_IN_2: now also U34.14 (A1)
- net DC_IN_3: now also U34.15 (A2)
- net DC_IN_4: now also U34.12 (A3)
- net DIN_1: now also U34.1 (A4)
- net DIN_2: now also U34.5 (A5)
- net DIN_3: now also U34.2 (A6)
- net DIN_4: now also U34.4 (A7)
Changed lines of the file:
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@@
+		)
+	)
+	(global_label "DIN_3"
+		(shape input)
+		(at 760.73 457.2 0)
+		(fields_autoplaced yes)
+		(effects
+			(font
+				(size 1 1)
+			)
+			(justify left)
+		)
+		(property "Intersheetrefs" "${INTERSHEET_REFS}"
+			(at 767.3184 457.2 0)
+			(effects
+				(font
+					(size 1 1)
+				)
+				(justify left)
+				(hide yes)
+			)
 		)
 	)
@@
 		)
 	)
+	(global_label "DC_IN_4"
+		(shape input)
+		(at 760.73 449.58 0)
+		(fields_autoplaced yes)
+		(effects
+			(font
+				(size 1 1)
+			)
+			(justify left)
+		)
+		(property "Intersheetrefs" "${INTERSHEET_REFS}"
+			(at 769.0803 449.58 0)
+			(effects
+				(font
+					(size 1 1)
+				)
+				(justify left)
+				(hide yes)
+			)
+		)
+	)
 	(global_label "VCOUPLER"
 		(shape input)
@@
 		)
 	)
+	(global_label "DIN_2"
+		(shape input)
+		(at 760.73 454.66 0)
+		(fields_autoplaced yes)
+		(effects
+			(font
+				(size 1 1)
+			)
+			(justify left)
+		)
+		(property "Intersheetrefs" "${INTERSHEET_REFS}"
+			(at 767.3184 454.66 0)
+			(effects
+				(font
+					(size 1 1)
+				)
+				(justify left)
+				(hide yes)
+			)
+		)
+	)
 	(global_label "V_DC_IN"
 		(shape input)
@@
 		)
 	)
+	(global_label "DC_IN_2"
+		(shape input)
+		(at 760.73 444.5 0)
+		(fields_autoplaced yes)
+		(effects
+			(font
+				(size 1 1)
+			)
+			(justify left)
+		)
+		(property "Intersheetrefs" "${INTERSHEET_REFS}"
+			(at 769.0803 444.5 0)
+			(effects
+				(font
+					(size 1 1)
+				)
+				(justify left)
+				(hide yes)
+			)
+		)
+	)
 	(global_label "MASTER_MODBUS_A"
 		(shape input)
@@
 		)
 	)
+	(global_label "DIN_1"
+		(shape input)
+		(at 760.73 452.12 0)
+		(fields_autoplaced yes)
+		(effects
+			(font
+				(size 1 1)
+			)
+			(justify left)
+		)
+		(property "Intersheetrefs" "${INTERSHEET_REFS}"
+			(at 767.3184 452.12 0)
+			(effects
+				(font
+					(size 1 1)
+				)
+				(justify left)
+				(hide yes)
+			)
+		)
+	)
 	(global_label "DOUT_DRV_2"
 		(shape input)
@@
 		)
 	)
+	(global_label "DC_IN_1"
+		(shape input)
+		(at 760.73 441.96 0)
+		(fields_autoplaced yes)
+		(effects
+			(font
+				(size 1 1)
+			)
+			(justify left)
+		)
+		(property "Intersheetrefs" "${INTERSHEET_REFS}"
+			(at 769.0803 441.96 0)
+			(effects
+				(font
+					(size 1 1)
+				)
+				(justify left)
+				(hide yes)
+			)
+		)
+	)
 	(global_label "DC_OUT_2_B"
 		(shape input)
@@
 		)
 	)
+	(global_label "DIN_4"
+		(shape input)
+		(at 760.73 459.74 0)
+		(fields_autoplaced yes)
+		(effects
+			(font
+				(size 1 1)
+			)
+			(justify left)
+		)
+		(property "Intersheetrefs" "${INTERSHEET_REFS}"
+			(at 767.3184 459.74 0)
+			(effects
+				(font
+					(size 1 1)
+				)
+				(justify left)
+				(hide yes)
+			)
+		)
+	)
 	(global_label "E_AIN_3"
 		(shape input)
@@
 				)
 				(justify left)
+				(hide yes)
+			)
+		)
+	)
+	(global_label "DC_IN_3"
+		(shape input)
+		(at 760.73 447.04 0)
+		(fields_autoplaced yes)
+		(effects
+			(font
+				(size 1 1)
+			)
+			(justify left)
+		)
+		(property "Intersheetrefs" "${INTERSHEET_REFS}"
+			(at 769.0803 447.04 0)
+			(effects
+				(font
+					(size 1 1)
+				)
+				(justify left)

Commit message: Done Schematic ESP32 PLC
Parts:
- removed C28, C29: 22uF, Capacitor_SMD:C_0603_1608Metric, symbol Device:C_Polarized
- removed C3, C4, C5, C6: 0.1uF, Capacitor_SMD:C_0402_1005Metric, symbol Device:C
- removed K1, K2, K3, K4: Y14x-1C-xxDS, Relay_THT:Relay_SPDT_HsinDa_Y14, symbol Relay:Y14x-1C-xxDS
- removed RV1, RV2, RV3, RV4: 20K, symbol Device:R_Potentiometer_US
- removed U17, U19, U20, U21: OP07, Package_SO:SOIC-8_3.9x4.9mm_P1.27mm, symbol Amplifier_Operational:OP07
- added C28, C29: 22uF, Capacitor_SMD:C_0603_1608Metric, symbol Device:C
- added JP11, JP12, JP13, JP14, JP15, JP16, JP17, JP18: SolderJumper_3_Open, Jumper:SolderJumper-3_P1.3mm_Open_Pad1.0x1.5mm, symbol Jumper:SolderJumper_3_Open
- added K1, K2, K3, K5: SANYOU_SRD_Form_C, Relay_THT:Relay_SPDT_SANYOU_SRD_Series_Form_C, symbol Relay:SANYOU_SRD_Form_C
- added R68, R72: 210K, Resistor_SMD:R_0402_1005Metric_Pad0.72x0.64mm_HandSolder, symbol Device:R
- added R69, R73: 200K, Resistor_SMD:R_0402_1005Metric_Pad0.72x0.64mm_HandSolder, symbol Device:R
- added R70, R74: 5.1K, Resistor_SMD:R_0402_1005Metric_Pad0.72x0.64mm_HandSolder, symbol Device:R
- added R71, R75, R76, R77, R78, R79: 4.7K, Resistor_SMD:R_0402_1005Metric_Pad0.72x0.64mm_HandSolder, symbol Device:R
- C22: now not fitted
- C23, C26: footprint Capacitor_SMD:C_0805_2012Metric_Pad1.18x1.45mm_HandSolder -> Capacitor_SMD:C_Elec_10x10.2; LCSC C15850 -> C28241; now not fitted
- C30, C31: footprint Capacitor_SMD:C_0805_2012Metric_Pad1.18x1.45mm_HandSolder -> Capacitor_SMD:C_0603_1608Metric; LCSC C15850 -> C59461
- D1, D2, D3, D4: value D -> 1N4001; footprint (none) -> Diode_SMD:D_SOD-123F; LCSC (none) -> C2892326
- D10, D12, D6, D7: value DIODE -> 1N4001
- D11, D13, D14, D16, D5, D8, D9: LCSC C2296 -> C2297
- J1, J2, J3, J4: footprint (none) -> TerminalBlock_Phoenix:TerminalBlock_Phoenix_MKDS-1,5-12-5.08_1x12_P5.08mm_Horizontal
- J9: footprint Connector_JST:JST_PH_B2B-PH-K_1x02_P2.00mm_Vertical -> Connector_PinHeader_2.54mm:PinHeader_1x02_P2.54mm_Vertical
- JP1, JP10, JP3, JP4, JP6, JP8: footprint (none) -> Jumper:SolderJumper-3_P1.3mm_Open_Pad1.0x1.5mm
- JP2: footprint (none) -> Jumper:SolderJumper-2_P1.3mm_Open_Pad1.0x1.5mm
- R1, R12, R6, R9: footprint (none) -> Resistor_SMD:R_0603_1608Metric_Pad0.98x0.95mm_HandSolder; LCSC (none) -> C25804
- R10, R11, R13, R14, R16, R18, R19, R2, R21, R22, R24, R3, R4, R5, R7, R8: footprint (none) -> Resistor_SMD:R_0603_1608Metric_Pad0.98x0.95mm_HandSolder; LCSC (none) -> C21190
- R15, R17, R20, R23: footprint Resistor_SMD:R_0603_1608Metric -> Resistor_SMD:R_0603_1608Metric_Pad0.98x0.95mm_HandSolder; LCSC C21190 -> C22975
- R25, R26, R27, R28, R29, R30, R31, R32, R33, R34, R35, R36, R37, R38, R39, R40, R49, R50, R51, R52, R53, R54, R55, R59, R60, R61, R67: footprint Resistor_SMD:R_0603_1608Metric -> Resistor_SMD:R_0603_1608Metric_Pad0.98x0.95mm_HandSolder
- R43, R47: value 5.1K -> 210K; LCSC C25905 -> C2686484
- R44, R48: value 4.7K -> 200K; LCSC C25900 -> C286555
- R66: LCSC C100703 -> C12447
- U1, U10, U11, U12, U13, U14, U15, U16, U2, U3, U4, U5, U6, U7, U8, U9: footprint Package_DIP:DIP-4_W7.62mm -> InnovKits:APC-817xx-SL_AMB; LCSC (none) -> C66405
- U18: footprint Package_SO:TSSOP-10_3x3mm_P0.5mm -> InnovKits:DGS0010A_L
- U28: footprint B_S-2WR2_MNS -> InnovKits:B_S-2WR2_MNS; LCSC (none) -> C5369473
- U34: footprint (none) -> Package_SO:SO-16_3.9x9.9mm_P1.27mm; LCSC (none) -> C9386
Connections:
- net 24VIN is gone; now on net +24V: J2.12 (Pin_12)
- net GND is gone; now on net GNDPWR: J2.7 (Pin_7), J2.8 (Pin_8), J2.9 (Pin_9), J4.6 (Pin_6)
- net SCL is gone; now on net SCL_E: J4.7 (Pin_7)
- net SDA is gone; now on net SDA_E: J4.8 (Pin_8)
- net +24V: now also K1.5, K2.5, K3.5, K5.5
- net +3.3V: now also R76.2, R77.2
- net +3.3VA: now also C29.2
- net +5VA: now also C28.2, R78.2, R79.2
- net ADC_IN_0: now also JP12.2 (C); no longer R41.2, R42.1
- net ADC_IN_1: now also JP14.2 (C); no longer R43.2, R44.1
- net ADC_IN_2: now also JP16.2 (C); no longer R45.2, R46.1
- net ADC_IN_3: now also JP18.2 (C); no longer R47.2, R48.1
- net DC_OUT_1_A: now also K5.1
- net DC_OUT_1_B: now also K5.3
- net DC_OUT_2_A: now also K1.1
- net DC_OUT_2_B: now also K1.3
- net DC_OUT_3_A: now also K2.1
- net DC_OUT_3_B: now also K2.3
- net DC_OUT_4_A: now also K3.1
- net DC_OUT_4_B: now also K3.3
- net ESP_SCL: now also R77.1
- net ESP_SDA: now also R76.1
- net E_AIN_1: now also JP11.2 (C)
- net E_AIN_2: now also JP13.2 (C)
- net E_AIN_3: now also JP15.2 (C)
- net E_AIN_4: now also JP17.2 (C)
- net GNDD: now also C30.1, C31.1, C32.1, C33.2, U31.1 (GND)
- net GNDPWR: now also C28.1, C29.1, R69.2, R71.2, R73.2, R75.2; no longer C30.1, C31.1, C32.1, C33.2, U31.1 (GND)
- net SCL_E: now also R79.1
- net SDA_E: now also R78.1
- net at D5.1 (K), D6.1 (K), Q6.3 (D): now also K5.2
- net at D11.1 (K), D12.1 (K), Q8.3 (D): now also K3.2
- net at R45.1: now also JP13.1 (A)
- net at D10.1 (K), D9.1 (K), Q7.3 (D): now also K2.2
- net at D7.1 (K), D8.1 (K), Q5.3 (D): now also K1.2
- net at R47.1: now also JP15.3 (B)
- net at R41.1: now also JP11.1 (A)
- net at R43.1: now also JP13.3 (B)
- new net: JP17.1 (A), R74.1
- new net: JP18.3 (B), R74.2, R75.1
- new net: JP15.1 (A), R70.1
- new net: JP16.3 (B), R70.2, R71.1
- new net: JP16.1 (A), R47.2, R48.1
- new net: JP18.1 (A), R72.2, R73.1
- new net: JP14.3 (B), R45.2, R46.1
- new net: JP11.3 (B), R68.1
- new net: JP17.3 (B), R72.1
- new net: JP12.1 (A), R68.2, R69.1
- new net: JP12.3 (B), R41.2, R42.1
- new net: JP14.1 (A), R43.2, R44.1
- no-connect marks 24 -> 38
Other:
- moved on the sheet: C1, C2, JP2, R41, R42, R49, U18, U22

Commit message: Started PCB Component Placement
To Do:

Double Check Footprint of ADS1115
Modularize Relay Control
Change Big Capacitors to SMD Capacitors
Parts:
- added C3: 10uF, Capacitor_SMD:C_0805_2012Metric_Pad1.18x1.45mm_HandSolder, symbol Device:C
- added C4: 0.1uF, Capacitor_SMD:C_0402_1005Metric, symbol Device:C
- J9: footprint Connector_PinHeader_2.54mm:PinHeader_1x02_P2.54mm_Vertical -> Connector_JST:JST_EH_B2B-EH-A_1x02_P2.50mm_Vertical
Connections:
- net +5V: now also C3.2, C4.2
- net GNDD: now also C3.1, C4.1
