File: Strobe_Light_LED_Signage/Strobe_Light_LED_Signage-backups/Strobe_Light_LED_Signage.kicad_pcb (KiCad board)
At the start: 2 copper layers, 100 x 80 mm, 137 parts, among them J1 Conn_01x04_Socket, J2 USB_B_Micro, J3 Conn_01x02_Socket, J4 Conn_01x02_Socket, J5 Conn_01x02_Socket, J6 Screw_Terminal_01x16, J7 Screw_Terminal_01x16, J8 Conn_01x02_Socket, J9 Conn_01x03_Socket, K1 EE2-5NU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

Commit message: Version 1.0 of both Strobe Light and PLC Done
Routing:
- net GND: vias 129 -> 257
Other:
- board size 100 x 80 mm -> 99.9 x 80.3 mm
